Commit message: limit bug fix in urdf; added joint_commander

File: ros packages/jlr23/urdf/jlr23.urdf (robot description, URDF)
Before this commit: robot jlr23, 9 links, 8 joints
Joints:
- joint camera_joint: limit lower=0 upper=0.71 effort=0 velocity=0 -> lower=0 upper=0.71 effort=1.2 velocity=1
- joint prismatic: limit lower=0 upper=0.71 effort=0 velocity=0 -> lower=0 upper=0.71 effort=80.0 velocity=1
- joint r1: limit lower=1.9 upper=6.08 effort=0 velocity=0 -> lower=1.9 upper=6.6 effort=1.2 velocity=1
- joint r2: limit lower=-3.14 upper=3.14 effort=0 velocity=0 -> lower=-31400 upper=31400 effort=1.2 velocity=1
- joint r3: limit lower=-3.14 upper=3.14 effort=0 velocity=0 -> lower=-31400 upper=31400 effort=1.2 velocity=1
- joint r4: limit lower=-1.82 upper=1.82 effort=0 velocity=0 -> lower=-1.82 upper=1.82 effort=1.2 velocity=1
- joint r5: limit lower=-3.14 upper=3.14 effort=0 velocity=0 -> lower=-31400 upper=31400 effort=1.2 velocity=1

Commit message: camera pose fix in urdf

File: ros packages/jlr23/urdf/jlr23.urdf (robot description, URDF)
Before this commit: robot jlr23, 9 links, 8 joints
Joints:
- joint camera_joint: origin xyz=0.12 0.1 -0.0125 rpy=1.5708 0 1.5708 -> xyz=0.015 0.1 -0.0125 rpy=1.5708 0 1.5708
- joint link_0_JOINT_0: origin xyz=0 0.025 0 rpy=0 -0 0 -> xyz=0 0 0 rpy=0 -0 0
